Commit message: Balance_controller + gazebo implementation
Unfixed Ricatti equation

File: src/robot_description/urdf/biped.urdf (robot description, URDF)
Before this commit: robot groupedurdf, 45 links, 44 joints
Links:
- removed link 0_25__id_bearing__0_5__od__0_188__wd__shielded_
- removed link 0_25__id_bearing__0_5__od__0_188__wd__shielded__1
- removed link 8108_8__x2_7b805316_x0__1
- removed link 8108_8__x2_7b805316_x0__1_1
- removed link 8108_8__x2_7b805316_x0__1_mirrored
- removed link lidar_a1m8
- removed link part_1
- removed link part_1_1
- removed link part_1_10
- removed link part_1_12
- removed link part_1_13
- removed link part_1_14
- removed link part_1_16
- removed link part_1_19
- removed link part_1_2
- removed link part_1_3
- removed link part_1_4
- removed link part_1_5
- removed link part_1_6
- removed link part_1_7
- removed link part_1_8
- removed link part_1_9
- removed link part_1_mirrored
- removed link part_1_mirrored_1
- removed link part_2
- removed link part_2_1
- removed link part_2_4
- removed link part_2_5
- removed link part_2_6
- removed link part_3
- removed link part_3_1
- removed link part_3_2
- removed link part_3_3
- removed link part_3_4
- removed link part_3__2__loop_closure
- removed link part_4
- removed link part_5
- removed link part_6
- removed link part_7
- removed link part_8
- removed link part_9
- removed link root
- removed link v5_x2_9a7152a876d6_x0_
- removed link v5_x2_9a7152a876d6_x0__1
- removed link v5_x2_9a7152a876d6_x0__mirrored
- added link base_link; visual box size=0.2858 0.2096 0.1365
- added link left_lower_leg; visual cylinder length=0.2311 radius=0.0127
- added link left_upper_leg; visual cylinder length=0.2311 radius=0.0127
- added link left_wheel; visual cylinder length=0.052 radius=0.105
- added link right_lower_leg; visual cylinder length=0.2311 radius=0.0127
- added link right_upper_leg; visual cylinder length=0.2311 radius=0.0127
- added link right_wheel; visual cylinder length=0.052 radius=0.105
Joints:
- removed joint fastened_1
- removed joint group_1_fastened_joint
- removed joint group_1_fastened_joint_1
- removed joint group_1_fastened_joint_2
- removed joint group_1_fastened_joint_3
- removed joint group_1_fastened_joint_4
- removed joint group_1_fastened_joint_5
- removed joint group_1_fastened_joint_6
- removed joint group_1_fastened_joint_7
- removed joint group_1_fastened_joint_8
- removed joint group_1_fastened_joint_9
- removed joint group_1_fastened_joint_loop_closure
- removed joint group_2_fastened_joint
- removed joint group_2_fastened_joint_1
- removed joint group_2_fastened_joint_2
- removed joint group_2_fastened_joint_3
- removed joint group_2_fastened_joint_4
- removed joint group_2_fastened_joint_5
- removed joint group_2_fastened_joint_6
- removed joint group_2_fastened_joint_7
- removed joint group_3_fastened_joint
- removed joint group_3_fastened_joint_1
- removed joint group_3_fastened_joint_2
- removed joint group_3_fastened_joint_3
- removed joint group_3_fastened_joint_4
- removed joint group_3_fastened_joint_5
- removed joint group_4_fastened_joint
- removed joint group_4_fastened_joint_1
- removed joint group_4_fastened_joint_2
- removed joint group_4_fastened_joint_3
- removed joint group_4_fastened_joint_4
- removed joint group_4_fastened_joint_5
- removed joint group_4_fastened_joint_6
- removed joint group_4_fastened_joint_7
- removed joint hanging_node_to_root_joint
- removed joint revolute_1
- removed joint revolute_2
- removed joint revolute_3
- removed joint revolute_3_1
- removed joint revolute_4
- removed joint revolute_4_1
- removed joint revolute_5
- removed joint revolute_5_1
- removed joint revolute_5_2
- added joint left_hip_joint: type revolute, parent base_link, child left_upper_leg, origin xyz=0 0.179 -0.0683 rpy=0 0 0, axis 0 1 0, limit lower=0.10 upper=1.24 effort=20 velocity=10
- added joint left_knee_joint: type revolute, parent left_upper_leg, child left_lower_leg, origin xyz=0 0 -0.2311 rpy=0 0 0, axis 0 1 0, limit lower=-2.4804 upper=0 effort=20 velocity=10, mimic joint=left_hip_joint multiplier=-2 offset=0
- added joint left_wheel_joint: type continuous, parent left_lower_leg, child left_wheel, origin xyz=0 0 -0.2311 rpy=0 0 0, axis 0 1 0
- added joint right_hip_joint: type revolute, parent base_link, child right_upper_leg, origin xyz=0 -0.179 -0.0683 rpy=0 0 0, axis 0 1 0, limit lower=0.10 upper=1.24 effort=20 velocity=10
- added joint right_knee_joint: type revolute, parent right_upper_leg, child right_lower_leg, origin xyz=0 0 -0.2311 rpy=0 0 0, axis 0 1 0, limit lower=-2.4804 upper=0 effort=20 velocity=10, mimic joint=right_hip_joint multiplier=-2 offset=0
- added joint right_wheel_joint: type continuous, parent right_lower_leg, child right_wheel, origin xyz=0 0 -0.2311 rpy=0 0 0, axis 0 1 0

File: src/robot_description/urdf/biped_sim.urdf (robot description, URDF)
Before this commit: robot biped, 5 links, 4 joints
Links:
- link base_link: mass 2.0 -> 4.1; geometry collision box size=0.286 0.210 0.137; visual box size=0.286 0.210 0.137
- link left_leg: mass 0.4 -> 0.5; geometry collision box size=0.04 0.04 0.257; visual box size=0.04 0.04 0.257
- link left_wheel: mass 0.3 -> 1.76; geometry collision cylinder length=0.052 radius=0.105; visual cylinder length=0.052 radius=0.105
- link right_leg: mass 0.4 -> 0.5; geometry collision box size=0.04 0.04 0.257; visual box size=0.04 0.04 0.257
- link right_wheel: mass 0.3 -> 1.76; geometry collision cylinder length=0.052 radius=0.105; visual cylinder length=0.052 radius=0.105
Joints:
- joint left_hip_joint: axis 0 1 0 -> (none); limit lower=-1.0 upper=1.0 effort=20 velocity=5 -> (none); origin xyz=0 0.1 -0.06 -> xyz=0 0.179 -0.0685; type revolute -> fixed
- joint left_wheel_joint: origin xyz=0 0 -0.18 -> xyz=0 0 -0.257
- joint right_hip_joint: axis 0 1 0 -> (none); limit lower=-1.0 upper=1.0 effort=20 velocity=5 -> (none); origin xyz=0 -0.1 -0.06 -> xyz=0 -0.179 -0.0685; type revolute -> fixed
- joint right_wheel_joint: origin xyz=0 0 -0.18 -> xyz=0 0 -0.257
