Commit message: Prismatic joints + leg kinematics
Awaiting lean control

File: src/robot_description/urdf/biped_sim.urdf (robot description, URDF)
Before this commit: robot biped, 5 links, 4 joints
Links:
- link left_leg: geometry collision box size=0.04 0.04 0.160; visual box size=0.04 0.04 0.160
- link right_leg: geometry collision box size=0.04 0.04 0.160; visual box size=0.04 0.04 0.160
Joints:
- joint left_hip_joint: axis (none) -> 0 0 -1; limit (none) -> lower=0.0 upper=0.302 effort=200.0 velocity=0.3; type fixed -> prismatic
- joint left_wheel_joint: origin xyz=0 0 -0.257 -> xyz=0 0 -0.160
- joint right_hip_joint: axis (none) -> 0 0 -1; limit (none) -> lower=0.0 upper=0.302 effort=200.0 velocity=0.3; type fixed -> prismatic
- joint right_wheel_joint: origin xyz=0 0 -0.257 -> xyz=0 0 -0.160
